Commit message: fix the mistake in xacro of mid360

File: urdf/livox_mid360.xacro (robot description, xacro)
@@ -58,5 +58,5 @@
     </gazebo>
   </xacro:macro>
-  <xacro:macro name="Livox_Mid40" params="visualize:=True name:=livox">
+  <xacro:macro name="Livox_Mid360" params="visualize:=True name:=livox">
     <link name="${name}_base">
       <xacro:null_inertial/>
@@ -84,5 +84,5 @@
     <xacro:Livox_Mid_gazebo_sensor name="${name}" visualize="${visualize}"/>
   </xacro:macro>
-    <xacro:Livox_Mid40 name="livox"/>
+    <xacro:Livox_Mid360 name="livox"/>
   <xacro:include filename="$(find livox_laser_simulation)/urdf/standardrobots_oasis300.xacro"/>
   <xacro:link_oasis name="oasis"/>
